Commit message: bicycle model spawning in gazebo

File: src/bicycle_description/urdf/robot.urdf.xacro (robot description, xacro)
@@ -1,9 +1,12 @@
 <?xml version="1.0"?>
 <robot name = "bicycle" xmlns:xacro="http://www.ros.org/wiki/xacro">
+    <xacro:include filename="inertial_macros.xacro"/>
     <xacro:property name = "base_length" value = "0.5"/>
     <xacro:property name = "base_width" value = "0.1"/>
     <xacro:property name = "base_height" value = "0.05"/>
     <xacro:property name = "wheel_radius" value = "0.05"/>
-    <xacro:property name = "wheel_length" value = "0.05"/>
+    <xacro:property name = "wheel_length" value = "0.1"/>
+    <xacro:property name = "cylinder_length" value = "0.1"/>
+    <xacro:property name = "cylinder_radius" value = "0.01"/>
     <material name="blue">
         <color rgba="0 0 0.5 1" />
@@ -27,4 +30,13 @@
             <material name = "blue"/>
         </visual>
+        <collision>
+            <geometry>
+                <box size = "${base_length} ${base_width} ${base_height}"/>
+            </geometry>
+            <origin xyz = "0 0 0"/>
+        </collision>
+        <xacro:inertial_box mass="0.01" x="0.5" y="0.1" z="0.05">
+            <origin xyz="0 0 0" rpy="0 0 0"/>
+        </xacro:inertial_box>
     </link>
     <link name = "front_wheel">
@@ -36,4 +48,13 @@
             <material name = "grey"/>
         </visual>
+        <collision>
+            <geometry>
+                <cylinder radius = "${wheel_radius}" length = "${wheel_length}"/>
+            </geometry>
+            <origin xyz = "0 0 0" rpy = "0 0 0"/>
+        </collision>
+        <xacro:inertial_cylinder mass="0.01" length="${wheel_length}" radius="${wheel_radius}">
+            <origin xyz = "0 0 0" rpy ="0 0 0"/>
+        </xacro:inertial_cylinder>
     </link>
     <link name = "rear_wheel">
@@ -45,25 +66,52 @@
             <material name = "grey"/>
         </visual>
+        <collision>
+            <geometry>
+                <cylinder radius = "${wheel_radius}" length = "${wheel_length}"/>
+            </geometry>
+            <origin xyz = "0 0 0" rpy = "0 0 0"/>
+        </collision>
+        <xacro:inertial_cylinder mass="0.01" length="${wheel_length}" radius="${wheel_radius}">
+            <origin xyz = "0 0 0" rpy ="0 0 0"/>
+        </xacro:inertial_cylinder>
     </link>
     <link name = "front_wheel_cylinder">
         <visual>
             <geometry>
-                <cylinder radius = "0.01" length = "${wheel_length}"/>
+                <cylinder radius = "0.01" length = "${cylinder_length}"/>
             </geometry>
             <origin xyz = "0 0 0" rpy = "0 0 0"/>
             <material name = "grey"/>
         </visual>
+        <collision>
+            <geometry>
+                <cylinder radius = "0.01" length = "${cylinder_length}"/>
+            </geometry>
+            <origin xyz = "0 0 0" rpy = "0 0 0"/>
+        </collision>
+        <xacro:inertial_cylinder mass="0.005" length="${cylinder_length}" radius="${cylinder_radius}">
+            <origin xyz = "0 0 0" rpy ="0 0 0"/>
+        </xacro:inertial_cylinder>
     </link>
     <link name = "rear_wheel_cylinder">
         <visual>
             <geometry>
-                <cylinder radius = "0.01" length = "${wheel_length}"/>
+                <cylinder radius = "0.01" length = "${cylinder_length}"/>
             </geometry>
             <origin xyz = "0 0 0" rpy = "0 0 0"/>
             <material name = "grey"/>
         </visual>
+        <collision>
+            <geometry>
+                <cylinder radius = "0.01" length = "${cylinder_length}"/>
+            </geometry>
+            <origin xyz = "0 0 0" rpy = "0 0 0"/>
+        </collision>
+        <xacro:inertial_cylinder mass="0.005" length="${cylinder_length}" radius="${cylinder_radius}">
+            <origin xyz = "0 0 0" rpy ="0 0 0"/>
+        </xacro:inertial_cylinder>
     </link>
     <joint name = "base_joint" type = "fixed">
-        <origin xyz = "0 0 0.15"/>
+        <origin xyz = "0 0 0.2"/>
         <parent link = "base_footprint"/>
         <child link = "base_link"/>

Commit message: joint names are changed

File: src/bicycle_description/urdf/robot.urdf.xacro (robot description, xacro)
@@ -117,5 +117,5 @@
         <child link = "base_link"/>
     </joint>
-    <joint name = "base_front_cylinder_joint" type = "continuous">
+    <joint name = "steering_joint" type = "continuous">
         <origin xyz = "${base_length/2 - wheel_radius} 0 -0.01" rpy = "0 0 0"/>
         <parent link = "base_link"/>
@@ -123,5 +123,5 @@
         <axis xyz = "0 0 1"/>
     </joint>
-    <joint name = "cylinder_front_wheel_joint" type = "continuous">
+    <joint name = "front_wheel_joint" type = "continuous">
         <origin xyz = "0 0 ${-wheel_radius-wheel_length/2}" rpy = "${pi/2} 0 0"/>
         <parent link = "front_wheel_cylinder"/>
@@ -134,5 +134,5 @@
         <child link = "rear_wheel_cylinder"/>
     </joint>
-    <joint name = "cylinder_rear_wheel_joint" type = "continuous">
+    <joint name = "rear_wheel_joint" type = "continuous">
         <origin xyz = "0 0 ${-wheel_radius-wheel_length/2}" rpy = "${pi/2} 0 0"/>
         <parent link = "rear_wheel_cylinder"/>

Commit message: gazebo controllers working

File: src/bicycle_description/urdf/robot.urdf.xacro (robot description, xacro)
@@ -2,4 +2,5 @@
 <robot name = "bicycle" xmlns:xacro="http://www.ros.org/wiki/xacro">
     <xacro:include filename="inertial_macros.xacro"/>
+    <xacro:include filename="ros2_control.xacro" />
     <xacro:property name = "base_length" value = "0.5"/>
     <xacro:property name = "base_width" value = "0.1"/>
@@ -54,5 +55,5 @@
             <origin xyz = "0 0 0" rpy = "0 0 0"/>
         </collision>
-        <xacro:inertial_cylinder mass="0.01" length="${wheel_length}" radius="${wheel_radius}">
+        <xacro:inertial_cylinder mass="1.0" length="${wheel_length}" radius="${wheel_radius}">
             <origin xyz = "0 0 0" rpy ="0 0 0"/>
         </xacro:inertial_cylinder>
@@ -72,5 +73,5 @@
             <origin xyz = "0 0 0" rpy = "0 0 0"/>
         </collision>
-        <xacro:inertial_cylinder mass="0.01" length="${wheel_length}" radius="${wheel_radius}">
+        <xacro:inertial_cylinder mass="1.0" length="${wheel_length}" radius="${wheel_radius}">
             <origin xyz = "0 0 0" rpy ="0 0 0"/>
         </xacro:inertial_cylinder>
@@ -117,9 +118,10 @@
         <child link = "base_link"/>
     </joint>
-    <joint name = "steering_joint" type = "continuous">
+    <joint name = "steering_joint" type = "revolute">
         <origin xyz = "${base_length/2 - wheel_radius} 0 -0.01" rpy = "0 0 0"/>
         <parent link = "base_link"/>
         <child link = "front_wheel_cylinder"/>
         <axis xyz = "0 0 1"/>
+        <limit lower="-0.4" upper="0.4" effort="100.0" velocity="0.0"/>
     </joint>
     <joint name = "front_wheel_joint" type = "continuous">
@@ -128,4 +130,5 @@
         <child link = "front_wheel"/>
         <axis xyz = "0 0 1"/>
+        <dynamics damping="0.5"/>
     </joint>
         <joint name = "base_rear_cylinder_joint" type = "fixed">
@@ -139,4 +142,24 @@
         <child link = "rear_wheel"/>
         <axis xyz = "0 0 1"/>
+        <dynamics damping="0.5"/>
     </joint>
+    <gazebo reference="base_link">
+        <material>Gazebo/Red</material>
+    </gazebo>
+        <!-- <gazebo>
+            <plugin name = "diff_drive" filename="libgazebo_ros_diff_drive.so">
+                <left_joint>rear_wheel_joint</left_joint>
+                <right_joint>front_wheel_joint</right_joint>
+                <wheel_seperation>0.1</wheel_seperation>
+                <wheel_diameter>0.1</wheel_diameter>
+                <max_wheel_torque>200</max_wheel_torque>
+                <max_wheel_acceleration>10</max_wheel_acceleration>
+                <odometry_frame>odom</odometry_frame>
+                <robot_base_frame>base_link</robot_base_frame>
+                <publish_odom>true</publish_odom>
+                <publish_odom_tf>true</publish_odom_tf>
+                <publish_wheel_transform>true</publish_wheel_transform>
+                <use_stamped_vel>true</use_stamped_vel>
+            </plugin>
+        </gazebo> -->
 </robot>

Commit message: controller configured is working

File: src/bicycle_description/urdf/robot.urdf.xacro (robot description, xacro)
@@ -55,5 +55,5 @@
             <origin xyz = "0 0 0" rpy = "0 0 0"/>
         </collision>
-        <xacro:inertial_cylinder mass="1.0" length="${wheel_length}" radius="${wheel_radius}">
+        <xacro:inertial_cylinder mass="0.01" length="${wheel_length}" radius="${wheel_radius}">
             <origin xyz = "0 0 0" rpy ="0 0 0"/>
         </xacro:inertial_cylinder>
@@ -73,5 +73,5 @@
             <origin xyz = "0 0 0" rpy = "0 0 0"/>
         </collision>
-        <xacro:inertial_cylinder mass="1.0" length="${wheel_length}" radius="${wheel_radius}">
+        <xacro:inertial_cylinder mass="0.01" length="${wheel_length}" radius="${wheel_radius}">
             <origin xyz = "0 0 0" rpy ="0 0 0"/>
         </xacro:inertial_cylinder>
@@ -130,5 +130,4 @@
         <child link = "front_wheel"/>
         <axis xyz = "0 0 1"/>
-        <dynamics damping="0.5"/>
     </joint>
         <joint name = "base_rear_cylinder_joint" type = "fixed">
@@ -142,5 +141,4 @@
         <child link = "rear_wheel"/>
         <axis xyz = "0 0 1"/>
-        <dynamics damping="0.5"/>
     </joint>
     <gazebo reference="base_link">

File: src/bicycle_description/urdf/ros2_control.xacro (robot description, xacro)
@@ -34,4 +34,14 @@
     </ros2_control>
     <gazebo>
+        <plugin name="p3d_base_controller" filename="libgazebo_ros_p3d.so">
+            <body_name>base_footprint</body_name>
+            <frame_name>world</frame_name>
+            <update_rate>30.0</update_rate>
+            <xyz_offset>0 0 0</xyz_offset>
+            <rpy_offset>0 0 0</rpy_offset>
+            <gaussian_noise>0.01</gaussian_noise>
+        </plugin>
+    </gazebo>
+    <gazebo>
         <plugin filename="libgazebo_ros2_control.so" name="gazebo_ros2_control">
             <parameters>$(find bicycle_description)/config/bicycle_controller.yaml</parameters>

Commit message: joint orientations corrected thus velocity commands corrected

File: src/bicycle_description/urdf/robot.urdf.xacro (robot description, xacro)
@@ -126,5 +126,5 @@
     </joint>
     <joint name = "front_wheel_joint" type = "continuous">
-        <origin xyz = "0 0 ${-wheel_radius-wheel_length/2}" rpy = "${pi/2} 0 0"/>
+        <origin xyz = "0 0 ${-wheel_radius-wheel_length/2}" rpy = "${-pi/2} 0 0"/>
         <parent link = "front_wheel_cylinder"/>
         <child link = "front_wheel"/>
@@ -137,5 +137,5 @@
     </joint>
     <joint name = "rear_wheel_joint" type = "continuous">
-        <origin xyz = "0 0 ${-wheel_radius-wheel_length/2}" rpy = "${pi/2} 0 0"/>
+        <origin xyz = "0 0 ${-wheel_radius-wheel_length/2}" rpy = "${-pi/2} 0 0"/>
         <parent link = "rear_wheel_cylinder"/>
         <child link = "rear_wheel"/>

Commit message: visualization for various cases implemented

File: src/bicycle_description/urdf/robot.urdf.xacro (robot description, xacro)
@@ -22,4 +22,7 @@
         <color rgba="0.5 0 0 1" />
     </material>
+    <material name = "white">
+        <color rgba = "1 1 1 0.5"/>
+    </material>
     <link name = "base_footprint"/>
     <link name = "base_link">
@@ -41,4 +44,18 @@
         </xacro:inertial_box>
     </link>
+    <link name = "base_visual">
+        <visual>
+            <geometry>
+                <box size = "5 3 ${base_height}"/>
+            </geometry>
+            <origin xyz = "0 0 0"/>
+            <material name = "white"/>
+        </visual>
+    </link>
+    <joint name = "vis_base" type = "fixed">
+        <origin xyz = "0 0 0"/>
+        <parent link = "base_link"/>
+        <child link = "base_visual"/>
+    </joint>
     <link name = "front_wheel">
         <visual>

Commit message: velocity is fed from a topic

File: src/bicycle_description/urdf/robot.urdf.xacro (robot description, xacro)
@@ -162,4 +162,14 @@
         <material>Gazebo/Red</material>
     </gazebo>
+    <!-- <gazebo reference="rear_wheel">
+        <material>Gazebo/Black</material>
+        <mu1 value="0.1"/>
+        <mu2 value="0.1"/>
+    </gazebo>
+    <gazebo reference="front_wheel">
+        <material>Gazebo/Black</material>
+        <mu1 value="0.1"/>
+        <mu2 value="0.1"/>
+    </gazebo> -->
     <!-- <gazebo reference="base_link">
         <sensor name="imu_sensor" type="imu">

Commit message: mpc done and working properly steering rate limit must be implemented

File: src/bicycle_description/urdf/robot.urdf.xacro (robot description, xacro)
@@ -47,5 +47,5 @@
         <visual>
             <geometry>
-                <box size = "5 3 ${base_height}"/>
+                <box size = "1 0.5 ${base_height}"/>
             </geometry>
             <origin xyz = "0 0 0"/>

Commit message: updated

File: src/bicycle_description/urdf/robot.urdf.xacro (robot description, xacro)
@@ -4,8 +4,8 @@
     <xacro:include filename="ros2_control.xacro" />
     <xacro:property name = "base_length" value = "0.5"/>
-    <xacro:property name = "base_width" value = "0.1"/>
+    <xacro:property name = "base_width" value = "0.2"/>
     <xacro:property name = "base_height" value = "0.05"/>
     <xacro:property name = "wheel_radius" value = "0.05"/>
-    <xacro:property name = "wheel_length" value = "0.1"/>
+    <xacro:property name = "wheel_length" value = "0.2"/>
     <xacro:property name = "cylinder_length" value = "0.1"/>
     <xacro:property name = "cylinder_radius" value = "0.01"/>
@@ -100,5 +100,5 @@
             </geometry>
             <origin xyz = "0 0 0" rpy = "0 0 0"/>
-            <material name = "grey"/>
+            <material name = "green"/>
         </visual>
         <collision>
@@ -118,5 +118,5 @@
             </geometry>
             <origin xyz = "0 0 0" rpy = "0 0 0"/>
-            <material name = "grey"/>
+            <material name = "green"/>
         </visual>
         <collision>
@@ -143,5 +143,5 @@
     </joint>
     <joint name = "front_wheel_joint" type = "continuous">
-        <origin xyz = "0 0 ${-wheel_radius-wheel_length/2}" rpy = "${-pi/2} 0 0"/>
+        <origin xyz = "0 0 ${-wheel_radius-wheel_length/4}" rpy = "${-pi/2} 0 0"/>
         <parent link = "front_wheel_cylinder"/>
         <child link = "front_wheel"/>
@@ -154,5 +154,5 @@
     </joint>
     <joint name = "rear_wheel_joint" type = "continuous">
-        <origin xyz = "0 0 ${-wheel_radius-wheel_length/2}" rpy = "${-pi/2} 0 0"/>
+        <origin xyz = "0 0 ${-wheel_radius-wheel_length/4}" rpy = "${-pi/2} 0 0"/>
         <parent link = "rear_wheel_cylinder"/>
         <child link = "rear_wheel"/>
@@ -164,11 +164,13 @@
     <!-- <gazebo reference="rear_wheel">
         <material>Gazebo/Black</material>
-        <mu1 value="0.1"/>
-        <mu2 value="0.1"/>
     </gazebo>
     <gazebo reference="front_wheel">
         <material>Gazebo/Black</material>
-        <mu1 value="0.1"/>
-        <mu2 value="0.1"/>
+    </gazebo>
+    <gazebo reference="front_wheel_cylinder">
+        <material>Gazebo/Blue</material>
+    </gazebo>
+    <gazebo reference="rear_wheel_cylinder">
+        <material>Gazebo/Blue</material>
     </gazebo> -->
     <!-- <gazebo reference="base_link">
